Commit message: replaced terrence urdf with a basic 4 wheel robot containing a lidar and camera. Gazebo implementation incomplete.

File: ros2/description/urdf/colors.xacro (robot description, xacro)
@@ -5,62 +5,12 @@
     <color rgba="1 0 0 1"/>
   </material>
-  <material name="green">
-    <color rgba="0 1 0 1"/>
-  </material>
   <material name="blue">
     <color rgba="0 0 1 1"/>
   </material>
-  <material name="yellow">
-    <color rgba="1 1 0 1"/>
+  <material name="gray">
+    <color rgba="0.6 0.6 0.6 1"/>
   </material>
-  <material name="cyan">
-    <color rgba="0 1 1 1"/>
-  </material>
-  <material name="magenta">
-    <color rgba="1 0 1 1"/>
-  </material>
-  <!-- Neutrals -->
-  <material name="white">
-    <color rgba="1 1 1 1"/>
-  </material>
-  <material name="black">
-    <color rgba="0 0 0 1"/>
-  </material>
-  <material name="gray">
-    <color rgba="0.5 0.5 0.5 1"/>
-  </material>
-  <material name="dark_gray">
-    <color rgba="0.25 0.25 0.25 1"/>
-  </material>
-  <!-- Extra fun colors -->
   <material name="orange">
     <color rgba="1 0.5 0 1"/>
   </material>
-  <material name="purple">
-    <color rgba="0.5 0 0.5 1"/>
-  </material>
-  <material name="pink">
-    <color rgba="1 0.75 0.8 1"/>
-  </material>
-  <material name="lime">
-    <color rgba="0.75 1 0 1"/>
-  </material>
-  <material name="teal">
-    <color rgba="0 0.5 0.5 1"/>
-  </material>
-  <material name="navy">
-    <color rgba="0 0 0.5 1"/>
-  </material>
-  <material name="brown">
-    <color rgba="0.6 0.3 0.1 1"/>
-  </material>
-  <material name="gold">
-    <color rgba="1 0.84 0 1"/>
-  </material>
-  <material name="silver">
-    <color rgba="0.75 0.75 0.75 1"/>
-  </material>
-  <material name="maroon">
-    <color rgba="0.5 0 0 1"/>
-  </material>
 </robot>

File: ros2/description/urdf/tootles.urdf.xacro (robot description, xacro)
@@ -1,380 +1,10 @@
 <?xml version="1.0" encoding="utf-8"?>
-<robot xmlns:xacro="http://www.ros.org/wiki/xacro" name="LilT_Combined_URDF">
-  <xacro:arg name="sim_mode" default="false"/>
-  <xacro:include filename="ros2_control.xacro"/>
-  <!-- COLORS -->
+<!-- You can name your robot whatever you like, but it *must* have a name! -->
+<robot name="Tootles" xmlns:xacro="http://www.ros.org/wiki/xacro">
   <xacro:include filename="colors.xacro"/>
-  <!-- LIDAR -->
-  <!-- Cant' use LiDAR anymore. If need reenabled, uncomment this and the roz_gz_bridge lidar-->
-  <!-- <xacro:include filename="lidar.xacro"/> -->
-  <!-- IMU -->
-  <xacro:include filename="imu.xacro"/>
-  <!-- CAMERA -->
-  <xacro:include filename="camera.xacro"/>
-  <link name="base_link" />
-  <link name="base_footprint" />
-  <joint name="base_joint" type="fixed">
-    <parent link="base_link" />
-    <child link="base_footprint" />
-    <origin xyz="0 0 0" rpy="0 0 0" />
-  </joint>
-  <!-- Base Link and Joint -->
-  <link name="Base">
-    <inertial>
-     <origin xyz="0.0071933 0.035942 -0.17341" rpy="0 0 0" />
-      <mass value="1.0994" />
-      <inertia ixx="0.0052099" ixy="-7.8944E-22" ixz="-4.9264E-20" iyy="0.0060071" iyz="3.293E-21"
-        izz="0.0014684" />
-    </inertial>
-    <visual>
-      <origin xyz="0 0 0" rpy="0 0 0" />
-      <geometry>
-        <mesh filename="file://$(find description)/meshes/Base.STL" />
-      </geometry>
-      <material name="teal">
-        <color rgba="0.75294 0.75294 0.75294 1" />
-      </material>
-    </visual>
-    <collision>
-      <origin xyz="0 0 0" rpy="0 0 0" />
-      <geometry>
-        <mesh filename="file://$(find description)/meshes/Base.STL" />
-      </geometry>
-    </collision>
-  </link>
-  <joint name="Baseplate_joint" type="fixed">
-    <origin xyz="0.136145 0 0" rpy="${pi/2} 0 ${pi/2}" />
-    <parent link="base_link" />
-    <child link="Base" />
-  </joint>
-  <gazebo reference="Base">
-    <material>Gazebo/White</material>
-  </gazebo>
-  <!-- Frictionless model of actual driver wheel (does drive the bot in the sim) s-->
-  <link name="DriverWheel">
-    <inertial>
-      <origin xyz="-0.030264 6.665E-05 1.2263E-10" rpy="0 0 0" />
-      <mass value="0.5" />
-      <inertia ixx="3.7938E-05" ixy="-6.4305E-20" ixz="-1.3428E-19" iyy="1.9406E-05"
-        iyz="2.6768E-13" izz="1.9256E-05" />
-    </inertial>
-    <visual>
-      <origin xyz="0 0 0" rpy="0 0 0" />
-      <geometry>
-        <mesh filename="file://$(find description)/meshes/DriverWheel.STL" />
-      </geometry>
-      <material name="green">
-        <color rgba="0.79216 0.81961 0.93333 1" />
-      </material>
-    </visual>
-    <collision>
-      <origin xyz="0 0 0" rpy="0 0 0" />
-      <geometry>
-        <!-- <mesh filename="file://$(find description)/meshes/DriverWheel.STL" /> -->
-        <sphere radius="0.05"/>
-      </geometry>
-    </collision>
-  </link>
-  <joint name="DW_Joint" type="fixed"> <origin xyz="0.17907 -0.0127 -0.0127" rpy="0 0 0" />
-    <parent link="Base" />
-    <child link="DriverWheel" />
-  </joint>
-  <gazebo reference="DriverWheel">
-    <material>Gazebo/Blue</material>
-      <!-- <mu1 value="0.001"/>
-      <mu2 value="0.001"/> -->
-      <mu1 value="0.0"/> <!-- ARE WE ALLOWED TO DO THIS??? -->
-      <mu2 value="0.0"/>
-      <!-- <kp value="10000000.0" />
-      <kd value="1.0" /> -->
-  </gazebo>
-  <!-- Rear Caster Driver Wheel and Joint -->
-  <link name="RearDriverWheel">
-    <inertial>
-      <origin xyz="-0.030264 6.665E-05 1.2263E-10" rpy="0 0 0" />
-      <mass value="0.5" />
-      <inertia ixx="3.7938E-05" ixy="-6.4305E-20" ixz="-1.3428E-19" iyy="1.9406E-05"
-        iyz="2.6768E-13" izz="1.9256E-05" />
-    </inertial>
-    <!-- use sprocket for visual (it wont spin unfortunately) -->
-    <visual>
-      <origin xyz="-0.0397 0 0" rpy="0 0 0" />
-      <geometry>
-        <mesh filename="file://$(find description)/meshes/DriverSprocket.STL" />
-      </geometry>
-      <material name="blue">
-        <color rgba="0.79216 0.81961 0.93333 1" />
-      </material>
-    </visual>
-    <collision>
-      <origin xyz="-0.030264 6.665E-05 1.2263E-10" rpy="0 0 0" />
-      <geometry>
-        <!-- <mesh filename="file://$(find description)/meshes/DriverWheel.STL" /> -->
-        <sphere radius="0.05"/>
-      </geometry>
-    </collision>
-  </link>
-  <joint name="RDW_Joint" type="fixed"> <origin xyz="0.17907 -0.0127 -0.25959" rpy="0 0 0" />
-    <parent link="Base" />
-    <child link="RearDriverWheel" />
-  </joint>
-  <gazebo reference="RearDriverWheel">
-    <material>Gazebo/Pink</material>
-      <!-- <mu1 value="0.001"/>
-      <mu2 value="0.001"/> -->
-      <mu1 value="0.0"/>
-      <mu2 value="0.0"/>
-      <!-- <kp value="10000000.0" />
-      <kd value="1.0" /> -->
-  </gazebo>
-  <!-- Invisible driver wheel that allows Tootles to turn accurately -->
-  <link name="DriverSprocket">
-    <inertial>
-      <origin xyz="0.0097746 -3.5292E-09 -5.2457E-08" rpy="0 0 0" />
-      <mass value="0.5" />
-      <inertia ixx="5.3673E-05" ixy="-1.8152E-12" ixz="1.8049E-14" iyy="2.7245E-05"
-        iyz="-1.9672E-11" izz="2.7245E-05" />
-    </inertial>
-    <!-- <visual>
-      <origin xyz="0 0 0" rpy="0 0 0" />
-      <geometry>
-        <mesh filename="file://$(find description)/meshes/DriverSprocket.STL" />
-      </geometry>
-      <material name="blue">
-        <color rgba="0.79216 0.81961 0.93333 1" />
-      </material>
-    </visual> -->
-    <collision>
-      <origin xyz="0 0 0" rpy="0 0 0" />
-      <geometry>
-        <!-- <mesh filename="file://$(find description)/meshes/DriverSprocket.STL" /> -->
-        <sphere radius="0.05"/>
-      </geometry>
-    </collision>
-  </link>
-  <joint name="DS_Joint" type="continuous">
-    <origin xyz="0.14605 -0.0127 -0.136145" rpy="0 0 0" />
-    <parent link="Base" />
-    <child link="DriverSprocket" />
-    <axis xyz="1 0 0" />
-    <limit effort="10" velocity="10" />
-  </joint>
-  <gazebo reference="DriverSprocket">
-    <material>Gazebo/Blue</material>
-  </gazebo>
-  <link name="PassWheel">
-    <inertial>
-      <origin xyz="0.020612 8.4006E-05 -0.00023239" rpy="0 0 0" />
-      <mass value="0.5" />
-      <inertia ixx="3.7938E-05" ixy="-6.4876E-20" ixz="-1.3466E-19" iyy="1.9406E-05"
-        iyz="-3.2644E-10" izz="1.9256E-05" />
-    </inertial>
-    <visual>
-      <origin xyz="0 0 0" rpy="0 0 0" />
-      <geometry>
-        <mesh filename="file://$(find description)/meshes/PassWheel.STL" />
-      </geometry>
-      <material name="purple">
-        <color rgba="0.79216 0.81961 0.93333 1" />
-      </material>
-    </visual>
-    <collision>
-      <origin xyz="0 0 0" rpy="0 0 0" />
-      <geometry>
-        <!-- <mesh filename="file://$(find description)/meshes/PassWheel.STL" /> -->
-        <sphere radius="0.05"/>
-      </geometry>
-    </collision>
-  </link>
-  <joint name="PW_Joint" type="fixed"> <origin xyz="-0.17907 -0.0127 -0.0127" rpy="0 0 0" />
-    <parent link="Base" />
-    <child link="PassWheel" />
-  </joint>
-  <gazebo reference="PassWheel">
-    <material>Gazebo/Blue</material>
-      <mu1 value="0.0"/>
-      <mu2 value="0.0"/>
-  </gazebo>
-  <!-- rear pass wheel -->
-  <link name="RearPassWheel">
-    <inertial>
-      <origin xyz="0.020612 8.4006E-05 -0.00023239" rpy="0 0 0" />
-      <mass value="0.5" />
-      <inertia ixx="3.7938E-05" ixy="-6.4876E-20" ixz="-1.3466E-19" iyy="1.9406E-05"
-        iyz="-3.2644E-10" izz="1.9256E-05" />
-    </inertial>
-    <!-- sprocket visual - again, it wont move -->
-    <visual>
-      <origin xyz="0.0397 0 0" rpy="0 0 0" />
-      <geometry>
-        <mesh filename="file://$(find description)/meshes/PassSprocket.STL" />
-      </geometry>
-      <material name="gray">
-        <color rgba="0.79216 0.81961 0.93333 1" />
-      </material>
-    </visual>
-    <collision>
-      <origin xyz="0.020612 8.4006E-05 -0.00023239" rpy="0 0 0" />
-      <geometry>
-        <!-- <mesh filename="file://$(find description)/meshes/PassWheel.STL" /> -->
-        <sphere radius="0.05"/>
-      </geometry>
-    </collision>
-  </link>
-  <joint name="RPW_Joint" type="fixed"> <origin xyz="-0.17907 -0.0127 -0.25959" rpy="0 0 0" />
-    <parent link="Base" />
-    <child link="RearPassWheel" />
-  </joint>
-  <gazebo reference="RearPassWheel">
-    <material>Gazebo/White</material>
-      <mu1 value="0.0"/>
-      <mu2 value="0.0"/>
-  </gazebo>
-  <link name="PassSprocket">
-    <inertial>
-      <origin xyz="-0.0056813 -3.6211E-09 -5.2434E-08" rpy="0 0 0" />
-      <mass value="0.5" />
-      <inertia ixx="5.3673E-05" ixy="-1.8152E-12" ixz="2.2008E-14" iyy="2.7245E-05"
-        iyz="-2.0018E-11" izz="2.7245E-05" />
-    </inertial>
-    <!-- <visual>
-      <origin xyz="0 0 0" rpy="0 0 0" />
-      <geometry>
-        <mesh filename="file://$(find description)/meshes/PassSprocket.STL" />
-      </geometry>
-      <material name="gray">
-        <color rgba="0.79216 0.81961 0.93333 1" />
-      </material>
-    </visual> -->
-    <collision>
-      <origin xyz="0 0 0" rpy="0 0 0" />
-      <geometry>
-        <!-- <mesh filename="file://$(find description)/meshes/PassSprocket.STL" /> -->
-        <sphere radius="0.05"/>
-      </geometry>
-    </collision>
-  </link>
-  <joint name="PS_Joint" type="continuous">
-    <origin xyz="-0.14605 -0.0127 -0.136145" rpy="0 0 0" />
-    <parent link="Base" />
-    <child link="PassSprocket" />
-    <axis xyz="1 0 0" />
-    <limit effort="10" velocity="10" />
-  </joint>
-  <gazebo reference="PassSprocket">
-    <material>Gazebo/Blue</material>
-  </gazebo>
-  <link name="Loader">
-    <inertial>
-      <origin xyz="-0.14124 -0.17161 0.14187" rpy="0 0 0" />
-      <mass value="1.4896" />
-      <inertia ixx="0.011793" ixy="-2.9875E-05" ixz="2.4692E-05" iyy="0.020991" iyz="0.0052507"
-        izz="0.024104" />
-    </inertial>
-    <visual>
-      <origin xyz="0 0 0" rpy="0 0 0" />
-      <geometry>
-        <mesh filename="file://$(find description)/meshes/Loader.STL" />
-      </geometry>
-      <material name="yellow">
-        <color rgba="1 0 0 1" />
-      </material>
-    </visual>
-    <collision>
-      <origin xyz="0 0 0" rpy="0 0 0" />
-      <geometry>
-        <mesh filename="file://$(find description)/meshes/Loader.STL" />
-      </geometry>
-    </collision>
-  </link>
-  <joint name="LoaderJoint" type="revolute">
-    <origin xyz="0.14135 0.20066 -0.03683" rpy="0 0 0" />
-    <parent link="Base" />
-    <child link="Loader" />
-    <axis xyz="-1 0 0" />
-    <limit lower="0" upper="1.571" effort="10" velocity="0.7854" />
-  </joint>
-  <gazebo reference="Loader">
-    <material>Gazebo/Red</material>
-    <mu1 value="0.001"/>
-    <mu2 value="0.001"/>
-  </gazebo>
-  <link name="Hopper">
-    <inertial>
-      <origin xyz="-0.079042 0.080085 0.065194" rpy="0 0 0" />
-      <mass value="0.29528" />
-      <inertia ixx="0.002494" ixy="3.9471E-05" ixz="3.2132E-05" iyy="0.0032471" iyz="-0.00071427"
-        izz="0.0022122" />
-    </inertial>
-    <visual>
-      <origin xyz="0 0 0" rpy="0 0 0" />
-      <geometry>
-        <mesh filename="file://$(find description)/meshes/Hopper.STL" />
-      </geometry>
-      <material name="pink">
-        <color rgba="0.79216 0.81961 0.93333 1" />
-      </material>
-    </visual>
-    <collision>
-      <origin xyz="0 0 0" rpy="0 0 0" />
-      <geometry>
-        <mesh filename="file://$(find description)/meshes/Hopper.STL" />
-      </geometry>
-    </collision>
-  </link>
-  <joint name="HopperJoint" type="revolute">
-    <origin xyz="0.076774 0.05207 -0.3429" rpy="0 0 0" />
-    <parent link="Base" />
-    <child link="Hopper" />
-    <axis xyz="-1 0 0" />
-    <limit lower="0" upper="0.785" effort="10" velocity="0.3927" />
-  </joint>
-  <gazebo reference="Hopper">
-    <material>Gazebo/White</material>
-  </gazebo>
-  <link name="Door">
-    <inertial>
-      <origin xyz="-0.09525 -0.062153 -0.013449" rpy="0 0 0" />
-      <mass value="0.067736" />
-      <inertia ixx="0.00011563" ixy="1.0111E-19" ixz="1.4928E-21" iyy="0.00020595" iyz="-1.1678E-05"
-        izz="0.00031894" />
-    </inertial>
-    <visual>
-      <origin xyz="0 0 0" rpy="0 0 0" />
-      <geometry>
-        <mesh filename="file://$(find description)/meshes/Door.STL" />
-      </geometry>
-      <material name="silver">
-        <color rgba="0.79216 0.81961 0.93333 1" />
-      </material>
-    </visual>
-    <collision>
-      <origin xyz="0 0 0" rpy="0 0 0" />
-      <geometry>
-        <mesh filename="file://$(find description)/meshes/Door.STL" />
-      </geometry>
-    </collision>
-  </link>
-  <joint name="DoorJoint" type="revolute">
-    <origin xyz="0.014539 0.1397 -0.033006" rpy="0 0 0" />
-    <parent link="Hopper" />
-    <child link="Door" />
-    <axis xyz="1 0 0" />
-    <limit lower="0" upper="0.3927" effort="0" velocity="0" />
-  </joint>
-  <gazebo reference="Door">
-    <material>Gazebo/White</material>
-  </gazebo>
-  <!-- Mimic joints don't work in New Gazebo because it's dumb and stupid -->
-  <!-- Mimic joints -->
-  <!-- <gazebo>
-    <plugin filename="gz-sim-mimic-joint-system" name="gz::sim::systems::MimicJoint">
-        <joint>DS_Joint</joint>
-        <mimicJoint>DW_Joint</mimicJoint>
-    </plugin>
-    <plugin filename="gz-sim-mimic-joint-system" name="gz::sim::systems::MimicJoint">
-        <joint>PS_Joint</joint>
-        <mimicJoint>PW_Joint</mimicJoint>
-    </plugin>
-  </gazebo> -->
+  <xacro:include filename="inertial_macros.xacro"/>
+  <xacro:include filename="tootles_core.xacro"/>
+  <xacro:include filename="sensors.xacro"/>
+  <!-- <xacro:include filename="gazebo.xacro"/> -->
+  <link name="base_link"></link>
 </robot>
