Commit message: Added Gazebo Simulation, but pointcloud orientation is messed up

File: ros2/description/urdf/gazebo.xacro (robot description, xacro)
@@ -1,3 +1,166 @@
 <?xml version="1.0" encoding="utf-8"?>
 <robot xmlns:xacro="http://www.ros.org/wiki/xacro">
+  <gazebo reference ="chassis_link">
+    <visual>
+      <material>
+        <specular>0.1 0.1 0.1 1</specular>
+      </material>
+    </visual>
+    <collision>
+      <surface>
+        <friction>
+          <ode>
+            <mu>1.0</mu>
+            <mu2>1.0</mu2>
+          </ode>
+        </friction>
+        <contact>
+          <ode>
+            <kp>10000000.0</kp>
+            <kd>1.0</kd>
+          </ode>
+        </contact>
+      </surface>
+    </collision>
+  </gazebo>
+  <gazebo reference="front_left_wheel_link">
+    <visual>
+      <material>
+        <specular>0.1 0.1 0.1 1</specular>
+      </material>
+    </visual>
+    <collision>
+      <surface>
+        <friction>
+          <ode>
+            <mu>1.0</mu>
+            <mu2>1.0</mu2>
+          </ode>
+        </friction>
+        <contact>
+          <ode>
+            <kp>10000000.0</kp>
+            <kd>1.0</kd>
+          </ode>
+        </contact>
+      </surface>
+    </collision>
+  </gazebo>
+  <gazebo reference="front_right_wheel_link">
+    <visual>
+      <material>
+        <specular>0.1 0.1 0.1 1</specular>
+      </material>
+    </visual>
+    <collision>
+      <surface>
+        <friction>
+          <ode>
+            <mu>1.0</mu>
+            <mu2>1.0</mu2>
+          </ode>
+        </friction>
+        <contact>
+          <ode>
+            <kp>10000000.0</kp>
+            <kd>1.0</kd>
+          </ode>
+        </contact>
+      </surface>
+    </collision>
+  </gazebo>
+  <gazebo reference="back_left_wheel_link">
+    <visual>
+      <material>
+        <specular>0.1 0.1 0.1 1</specular>
+      </material>
+    </visual>
+    <collision>
+      <surface>
+        <friction>
+          <ode>
+            <mu>1.0</mu>
+            <mu2>1.0</mu2>
+          </ode>
+        </friction>
+        <contact>
+          <ode>
+            <kp>10000000.0</kp>
+            <kd>1.0</kd>
+          </ode>
+        </contact>
+      </surface>
+    </collision>
+  </gazebo>
+  <gazebo reference="back_right_wheel_link">
+    <visual>
+      <material>
+        <specular>0.1 0.1 0.1 1</specular>
+      </material>
+    </visual>
+    <collision>
+      <surface>
+        <friction>
+          <ode>
+            <mu>1.0</mu>
+            <mu2>1.0</mu2>
+          </ode>
+        </friction>
+        <contact>
+          <ode>
+            <kp>10000000.0</kp>
+            <kd>1.0</kd>
+          </ode>
+        </contact>
+      </surface>
+    </collision>
+  </gazebo>
+  <gazebo reference="lidar_link">
+    <material>Gazebo/Red</material>
+    <sensor name="laser" type="gpu_lidar">
+      <always_on>true</always_on>
+      <pose>0 0 0 0 0 0</pose>
+      <visualize>true</visualize>
+      <update_rate>10</update_rate>
+      <lidar>
+        <scan>
+          <horizontal>
+            <samples>360</samples>
+            <resolution>1</resolution>
+            <min_angle>-3.14</min_angle>
+            <max_angle>3.14</max_angle>
+          </horizontal>
+        </scan>
+        <range>
+          <min>0.3</min>
+          <max>12</max>
+        </range>
+      </lidar>
+      <topic>scan</topic>
+      <gz_frame_id>lidar_link</gz_frame_id>
+    </sensor>
+  </gazebo>
+  <gazebo reference="camera_link">
+    <material>Gazebo/Red</material>
+    <sensor name="rgbd_camera" type="rgbd_camera">
+      <pose> 0 0 0 0 0 0 </pose>
+      <visualize>true</visualize>
+      <update_rate>10</update_rate>
+      <camera>
+        <camera_info_topic>camera/camera_info</camera_info_topic>
+        <horizontal_fov>1.089</horizontal_fov>
+        <image>
+          <format>R8G8B8</format>
+          <width>640</width>
+          <height>480</height>
+        </image>
+        <clip>
+          <near>0.05</near>
+          <far>8.0</far>
+        </clip>
+      </camera>
+      <topic>camera</topic>
+      <gz_frame_id>camera_link_optical</gz_frame_id>
+    </sensor>
+  </gazebo>
 </robot>

File: ros2/description/urdf/sensors.xacro (robot description, xacro)
@@ -45,9 +45,9 @@
     </xacro:inertial_box>
   </link>
-  <!-- <joint name="camera_optical_joint" type="fixed">
+  <joint name="camera_optical_joint" type="fixed">
     <parent link="camera_link" />
     <child link="camera_link_optical" />
     <origin xyz="0 0 0" rpy="${-pi/2} 0 ${-pi/2}" />
   </joint>
-  <link name="camera_link_optical"></link> -->
+  <link name="camera_link_optical"></link>
 </robot>

File: ros2/description/urdf/tootles.urdf.xacro (robot description, xacro)
@@ -6,5 +6,5 @@
   <xacro:include filename="tootles_core.xacro"/>
   <xacro:include filename="sensors.xacro"/>
-  <!-- <xacro:include filename="gazebo.xacro"/> -->
+  <xacro:include filename="gazebo.xacro"/>
   <link name="base_link"></link>
 </robot>
