Commit message: added foxglove studio to launch file and renamed laser link/joint to lidar

File: ros2/description/urdf/sensors.xacro (robot description, xacro)
@@ -2,10 +2,10 @@
 <robot xmlns:xacro="http://www.ros.org/wiki/xacro">
   <!-- 2D LiDAR -->
-  <joint name="laser_joint" type="fixed">
+  <joint name="lidar_joint" type="fixed">
     <parent link="chassis_link" />
-    <child link="laser_link" />
+    <child link="lidar_link" />
     <origin xyz="0 0 0.1" rpy="0 0 0" />
   </joint>
-  <link name="laser_link">
+  <link name="lidar_link">
     <visual>
       <geometry>

Commit message: added collison and inertia to camera box, updated length of lidar cylinder

File: ros2/description/urdf/sensors.xacro (robot description, xacro)
@@ -10,5 +10,5 @@
     <visual>
       <geometry>
-        <cylinder length="0.05" radius="0.04" />
+        <cylinder length="0.05" radius="0.05" />
       </geometry>
       <material name="red" />
@@ -16,8 +16,8 @@
     <collision>
       <geometry>
-        <cylinder length="0.05" radius="0.04" />
+        <cylinder length="0.05" radius="0.05" />
       </geometry>
     </collision>
-    <xacro:inertial_cylinder mass="0.1" radius="0.04" length="0.05">
+    <xacro:inertial_cylinder mass="0.1" radius="0.05" length="0.05">
       <origin xyz="0 0 0" rpy="0 0 0" />
     </xacro:inertial_cylinder>
@@ -36,4 +36,12 @@
       <material name="orange" />
     </visual>
+    <collision>
+      <geometry>
+        <box size="0.4 0.3 0.15"/>
+      </geometry>
+    </collision>
+    <xacro:inertial_box mass="0.5" x="0.4" y = "0.3" z="0.15">
+      <origin xyz="0 0 0" rpy="0 0 0"/>
+    </xacro:inertial_box>
   </link>
   <!-- <joint name="camera_optical_joint" type="fixed">

Commit message: updated collison and inertia values for camera box

File: ros2/description/urdf/sensors.xacro (robot description, xacro)
@@ -38,8 +38,8 @@
     <collision>
       <geometry>
-        <box size="0.4 0.3 0.15"/>
+        <box size="0.010 0.03 0.03"/>
       </geometry>
     </collision>
-    <xacro:inertial_box mass="0.5" x="0.4" y = "0.3" z="0.15">
+    <xacro:inertial_box mass="0.01" x="0.010" y = "0.03" z="0.03">
       <origin xyz="0 0 0" rpy="0 0 0"/>
     </xacro:inertial_box>

Commit message: Get mujoco to launch with robot!!!

File: ros2/description/urdf/sensors.xacro (robot description, xacro)
@@ -2,5 +2,5 @@
 <robot xmlns:xacro="http://www.ros.org/wiki/xacro">
   <!-- 2D LiDAR -->
-  <joint name="lidar_joint" type="fixed">
+  <!-- <joint name="lidar_joint" type="fixed">
     <parent link="chassis_link" />
     <child link="lidar_link" />
@@ -22,5 +22,5 @@
       <origin xyz="0 0 0" rpy="0 0 0" />
     </xacro:inertial_cylinder>
-  </link>
+  </link> -->
   <!-- RGBD Camera -->
   <joint name="camera_joint" type="fixed">

Commit message: Add back sensors

File: ros2/description/urdf/sensors.xacro (robot description, xacro)
@@ -2,5 +2,5 @@
 <robot xmlns:xacro="http://www.ros.org/wiki/xacro">
   <!-- 2D LiDAR -->
-  <!-- <joint name="lidar_joint" type="fixed">
+  <joint name="lidar_joint" type="fixed">
     <parent link="chassis_link" />
     <child link="lidar_link" />
@@ -22,5 +22,5 @@
       <origin xyz="0 0 0" rpy="0 0 0" />
     </xacro:inertial_cylinder>
-  </link> -->
+  </link>
   <!-- RGBD Camera -->
   <joint name="camera_joint" type="fixed">
