Commit message: Fix range finders

File: ros2/description/urdf/mujoco_inputs.xacro (robot description, xacro)
@@ -35,5 +35,5 @@
       <!-- angle_increment rotated about the replicate frame's Y axis. The hardware intercface then combines -->
       <!-- them into a single LaserScan message. -->
-      <lidar ref_site="lidar_link" sensor_name="rf" min_angle="-0.3" max_angle="0.3" angle_increment="0.025" />
+      <lidar ref_site="lidar_link_optical" sensor_name="rf" min_angle="-0.3" max_angle="0.3" angle_increment="0.025" />
       <!-- The element with the type and name as listed below will be modified with the remaining attributes -->
       <!-- If the attribute already existed, it will be overwritten -->

File: ros2/description/urdf/sensors.xacro (robot description, xacro)
@@ -23,4 +23,10 @@
     </xacro:inertial_cylinder>
   </link>
+  <joint name="lidar_optical_joint" type="fixed">
+    <parent link="lidar_link" />
+    <child link="lidar_link_optical" />
+    <origin xyz="0.05 0 0" rpy="0 0 0" />
+  </joint>
+  <link name="lidar_link_optical"></link>
   <!-- RGBD Camera -->
   <joint name="camera_joint" type="fixed">
